File: blackmagic_richardeoin.sch (EAGLE design)
At the start: 52 parts, among them IC1 STM32F_48PIN, IC2 TXS0108, IC3 TLV70033DCK, IC4 IP4220CZ6, IC5 IP4220CZ6, Q1 IRLML5103, U1 AD8655ARMZ, U3 LT1763CDEPBF

Commit message: Update parts list with 2x esd, split passives into separte list for clarity
Connections:
- new net IC8: C8.P$1, U$41.VCC
- net 3.3V: no longer C8.P$1, U$41.VCC
Changed lines of the file:
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@@
-</segment>
-<segment>
-<pinref part="U$41" gate="A" pin="VCC"/>
-<pinref part="C8" gate="G$1" pin="P$1"/>
-<wire x1="2.54" y1="104.14" x2="2.54" y2="101.6" width="0.1524" layer="91"/>
-<pinref part="U$44" gate="G$1" pin="3.3V"/>
-<wire x1="2.54" y1="109.22" x2="2.54" y2="104.14" width="0.1524" layer="91"/>
-<wire x1="2.54" y1="104.14" x2="10.16" y2="104.14" width="0.1524" layer="91"/>
-<junction x="2.54" y="104.14"/>
 </segment>
 <segment>
@@
 </segment>
 </net>
+<net name="IC8" class="0">
+<segment>
+<pinref part="U$41" gate="A" pin="VCC"/>
+<pinref part="C8" gate="G$1" pin="P$1"/>
+<wire x1="2.54" y1="104.14" x2="2.54" y2="101.6" width="0.1524" layer="91"/>
+<pinref part="U$44" gate="G$1" pin="3.3V"/>
+<wire x1="2.54" y1="109.22" x2="2.54" y2="104.14" width="0.1524" layer="91"/>
+<wire x1="2.54" y1="104.14" x2="10.16" y2="104.14" width="0.1524" layer="91"/>
+<junction x="2.54" y="104.14"/>
+</segment>
+</net>
